File: elektronika/combat/combat.kicad_pcb (KiCad board)
At the start: 2 copper layers, 76 x 50 mm, 35 parts, among them J1 odbiornik, J2 naped_prawy, J3 naped_lewy, J4 buzzer, J5 wyjscie do silnika +-, J6 Conn_02x04_Odd_Even, J7 zasilanie xt30, J8 Conn_01x01_Pin, J800 USB_C_Receptacle_USB2.0_16P, U1 ESP32-S3-WROOM-1, U2 kontroler_bldc, U3 AMS1117, U4 przetwornica

Commit message: pcb wersja 2.0
Parts:
- H1, H2, H3, H4: footprint MountingHole:MountingHole_3.2mm_M3 -> MountingHole:MountingHole_3.2mm_M3_Pad_Via
- J6: value Conn_02x04_Odd_Even -> programator od adama wasa
- R1, R2: footprint PCM_SparkFun-Resistor:R_0603_1608Metric -> Resistor_SMD:R_0603_1608Metric
- moved D1 78.4 mm to (74.0, 107.5), turned to -90 degrees
- moved C2 65.0 mm to (77.8, 116.4), turned to 90 degrees
- moved U3 61.0 mm to (84.0, 111.7), turned to 180 degrees
- moved R6 60.5 mm to (85.5, 117.0)
- moved D3 56.7 mm to (91.0, 116.8), turned to 180 degrees
- moved C1 56.5 mm to (91.0, 109.5), turned to 90 degrees
- moved R1 54.3 mm to (89.7, 113.2), turned to -90 degrees
- moved J6 53.8 mm to (133.8, 143.9), turned to -90 degrees
- moved J4 53.3 mm to (102.7, 144.6), turned to 0 degrees
- moved U2 51.3 mm to (137.1, 130.6)
- moved D2 50.0 mm to (79.8, 107.0), turned to 0 degrees
- moved R2 49.1 mm to (92.0, 113.2), turned to 90 degrees
- moved J3 44.6 mm to (98.2, 103.0)
- moved J2 44.5 mm to (111.2, 103.0)
- moved J8 43.4 mm to (137.5, 102.8)
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Connections:
- J4 pad 1: GPIO1 -> GPI42
- J6 pad 2: RX -> R
- J6 pad 7: TX -> T
- TB1 pad 10: GPIO2 -> GPIO9
- TB1 pad 11: GPIO1 -> GPIO10
- TB1 pad 12: GPIO41 -> GPIO11
- TB1 pad 14: GPIO40 -> GPIO12
- TB1 pad 15: GPIO39 -> GPIO13
- TB1 pad 16: GPIO38 -> GPIO14
- U1 pad 17: unconnected-(U1-GPIO9/TOUCH9/ADC1_CH8/FSPIHD/SUBSPIHD-Pad17) -> GPIO9
- U1 pad 18: unconnected-(U1-GPIO10/TOUCH10/ADC1_CH9/FSPICS0/FSPIIO4/SUBSPICS0-Pad18) -> GPIO10
- U1 pad 19: unconnected-(U1-GPIO11/TOUCH11/ADC2_CH0/FSPID/FSPIIO5/SUBSPID-Pad19) -> GPIO11
- U1 pad 20: unconnected-(U1-GPIO12/TOUCH12/ADC2_CH1/FSPICLK/FSPIIO6/SUBSPICLK-Pad20) -> GPIO12
- U1 pad 21: unconnected-(U1-GPIO13/TOUCH13/ADC2_CH2/FSPIQ/FSPIIO7/SUBSPIQ-Pad21) -> GPIO13
- U1 pad 22: unconnected-(U1-GPIO14/TOUCH14/ADC2_CH3/FSPIWP/FSPIDQS/SUBSPIWP-Pad22) -> GPIO14
- U1 pad 23: GPIO21 -> ePWM
- U1 pad 24: unconnected-(U1-GPIO47/SPICLK_P/SUBSPICLK_P_DIFF-Pad24) -> GPIO21
- U1 pad 31: GPIO38 -> unconnected-(U1-GPIO38/FSPIWP/SUBSPIWP-Pad31)
- U1 pad 32: GPIO39 -> unconnected-(U1-MTCK/GPIO39/CLK_OUT3/SUBSPICS1-Pad32)
- U1 pad 33: GPIO40 -> unconnected-(U1-MTDO/GPIO40/CLK_OUT2-Pad33)
- U1 pad 34: GPIO41 -> unconnected-(U1-MTDI/GPIO41/CLK_OUT1-Pad34)
- U1 pad 35: GPIO1 -> GPI42
- U1 pad 36: unconnected-(U1-U0RXD/GPIO44/CLK_OUT2-Pad36) -> T
- U1 pad 37: unconnected-(U1-U0TXD/GPIO43/CLK_OUT1-Pad37) -> R
- U1 pad 38: GPIO2 -> unconnected-(U1-GPIO2/TOUCH2/ADC1_CH1-Pad38)
- U1 pad 39: GPIO1 -> unconnected-(U1-GPIO1/TOUCH1/ADC1_CH0-Pad39)
- U1 pad 4: ePWM -> unconnected-(U1-GPIO4/TOUCH4/ADC1_CH3-Pad4)
Routing:
- net R: track 0.00 -> 74.8 mm, vias 0 -> 2
- net T: track 0.00 -> 62.3 mm, vias 0 -> 2
- net (no net): track 45.5 -> 0.00 mm, vias 1 -> 0
- net GPIO14: track 0.00 -> 30.3 mm
- net GPIO13: track 0.00 -> 27.3 mm
- net B01: track 50.3 -> 25.2 mm
- net GPIO12: track 0.00 -> 24.2 mm
- net RX: track 40.0 -> 16.4 mm, vias 3 -> 2
- net USB.D-: track 29.3 -> 6.30 mm, vias 2 -> 0
- net EN: track 32.5 -> 9.87 mm, vias 4 -> 0
- net GPIO0: track 33.9 -> 11.5 mm
- net USB.D+: track 27.2 -> 6.38 mm, vias 2 -> 0
- net B02: track 43.5 -> 24.2 mm
- net GPIO11: track 0.00 -> 18.6 mm
- net A02: track 38.8 -> 22.0 mm
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- added copper zone on F.Cu, net Net-(J8-Pin_1)
- removed copper zone on F.Cu, net 11.1V
- removed copper zone on B.Cu, net GND
- removed copper zone on F.Cu, net GND
Other:
- board text added: "11.1V->5V"
- board text added: "12.08.2026 COMBAT1FUNT"
- board text added: "ADAM CETNER"
- board text added: "BROŃ"
- board text added: "ELRS NANO"
- board text added: "ESCBLDC"
- board text added: "ESP32WROOMS3"
- board text added: "KONAR"
- board text added: "LEWY"
- board text added: "MISTRZOWIE OD ELEKTRONIKI: MICHAŁ SADECKI WOJCIECH SZAFRAŃSKI"
- board text added: "MOSTEK H"
- board text added: "PRAWY"
- board text added: "USB_C"
- board text added: "ZASILANIE"
- board text removed: "+"
- board text removed: "-"
