File: elektronika/combat/combat.kicad_pcb (KiCad board)
At the start: 2 copper layers, 76 x 50 mm, 35 parts, among them J1 odbiornik, J2 naped_prawy, J3 naped_lewy, J4 buzzer, J5 wyjscie do silnika +-, J6 programator od adama wasa, J7 zasilanie xt30, J8 Conn_01x01_Pin, J800 USB_C_Receptacle_USB2.0_16P, U1 ESP32-S3-WROOM-1, U2 kontroler_bldc, U3 AMS1117, U4 przetwornica

Commit message: Pcb wersaj 2.2
Parts:
- H3, H4: moved to B.Cu
- moved R6 13.3 mm to (98.6, 114.4)
- moved D3 9.85 mm to (100.8, 116.4)
- moved S1 0.92 mm to (94.8, 113.8)
- moved H3 0.28 mm to (75.7, 102.7), turned to 180 degrees
- moved H2 0.28 mm to (144.3, 102.7)
- moved H4 0.28 mm to (75.7, 145.3), turned to 180 degrees
- moved H1 0.28 mm to (144.3, 145.3)
Routing:
- net GPI42: track 0.00 -> 40.4 mm, vias 0 -> 4
- net 11.1V: track 70.2 -> 81.1 mm
- net GND: track 0.00 -> 2.72 mm, vias 31 -> 25
- net Net-(D3-A): track 3.89 -> 2.26 mm
- net Net-(J800-CC2): track 12.9 -> 13.6 mm
- net +5V: track 79.8 -> 80.5 mm
- net GPIO0: track 11.5 -> 12.1 mm
- net R: track 74.8 -> 75.4 mm
- added copper zone on B.Cu, net GND

Commit message: dostosowano reguly do jlcpcb
Parts:
- C1: footprint Capacitor_SMD:C_0805_2012Metric_Pad1.18x1.45mm_HandSolder -> Capacitor_SMD:C_0603_1608Metric_Pad1.08x0.95mm_HandSolder
Connections:
- H1 pad 1: GND -> (no net)
- H2 pad 1: GND -> (no net)
- H3 pad 1: GND -> (no net)
- H4 pad 1: GND -> (no net)
Routing:
- net R: track 75.4 -> 83.4 mm, vias 2 -> 3
- net T: track 62.5 -> 66.2 mm
- net RX: track 16.4 -> 19.2 mm
- net TX: track 16.2 -> 18.2 mm
- net +5V: track 80.5 -> 81.6 mm
- net Net-(J800-CC2): track 13.6 -> 14.7 mm
